Commit message: 0_o

File: hydrone_aerial_underwater_description/urdf/hydrone_aerial_underwater.gazebo.xacro (robot description, xacro)
@@ -6,17 +6,22 @@
     assume NWU (otherwise cob is below cog?).
     -->
-    <xacro:property name="cob" value="0.0 0.0 0.0"/>
+    <xacro:property name="cob" value="0.0 0.0 0.3"/>
     <!-- Volume, see p.31 in Berg2012 -->
-    <!-- <xacro:property name="volume" value="1.83826"/> -->
-    <xacro:property name="volume" value="0.00142887 "/>
+    <xacro:property name="volume" value="1.83826"/>
+    <!-- <xacro:property name="volume" value="0.00142887 "/> -->
     <xacro:macro name="hydrone_aerial_underwater_hydro_model" params="namespace">
         <link name="${namespace}/base_link">
             <neutrally_buoyant>0</neutrally_buoyant>
             <volume>${volume}</volume>
+            <box>
+                <width>1.5</width>
+                <length>2.6</length>
+                <height>1.6</height>
+            </box>
             <center_of_buoyancy>${cob}</center_of_buoyancy>
             <hydrodynamic_model>
                 <type>fossen</type>
                 <!-- Added mass: see p.28 in Berg2012 -->
-                <!-- <added_mass>
+                <added_mass>
                      779.79 -6.8773 -103.32  8.5426 -165.54 -7.8033
                     -6.8773    1222   51.29  409.44 -5.8488  62.726
@@ -25,5 +30,5 @@
                     -165.54 -5.8488 -386.42 -10.027  842.69 -1.1162
                     -7.8033  62.726  10.775  21.019 -1.1162  224.32
-                </added_mass> -->
+                </added_mass>
                 <!-- <added_mass>
                      77.979 -0.68773 -10.332  0.85426 -16.554 -0.78033
@@ -34,5 +39,5 @@
                     -0.78033  6.2726  1.0775  2.1019 -0.11162  22.432
                 </added_mass> -->
-                <added_mass>
+                <!-- <added_mass>
                      0.77979 -0.0068773 -0.10332  0.00085426 -0.16554 -0.00078033
                     -0.0068773    1.222   0.05129  0.40944 -0.0058488  0.062726
@@ -41,19 +46,19 @@
                     -0.16554 -0.0058488 -0.38642 -0.010027  0.84269 -0.0011162
                     -0.078033  0.062726  0.010775  0.021019 -0.0011162  0.22432
-                </added_mass>
+                </added_mass> -->
                 <!-- Linear damping: see p.31 in Berg2012 -->
+                <linear_damping>
+                    -74.82 -69.48 -728.4 -268.8 -309.77 -105
+                </linear_damping>
                 <!-- <linear_damping>
-                    -74.82 -69.48 -728.4 -268.8 -309.77 -105
+                    -0.07482 -0.06948 -0.7284 -0.2688 -0.30977 -0.105
                 </linear_damping> -->
-                <linear_damping>
-                    -0.07482 -0.06948 -0.7284 -0.2688 -0.30977 -0.105
-                </linear_damping>
                 <!-- Non-linear damping: see p.30 in Berg2012 -->
+                <quadratic_damping>
+                    -748.22 -992.53 -1821.01 -672 -774.44 -523.27
+                </quadratic_damping>
                 <!-- <quadratic_damping>
-                    -748.22 -992.53 -1821.01 -672 -774.44 -523.27
+                    -0.74822 -0.99253 -1.82101 -0.672 -0.77444 -0.52327
                 </quadratic_damping> -->
-                <quadratic_damping>
-                    -0.74822 -0.99253 -1.82101 -0.672 -0.77444 -0.52327
-                </quadratic_damping>
             </hydrodynamic_model>
         </link>

File: hydrone_aerial_underwater_description/urdf/hydrone_aerial_underwater_base.xacro (robot description, xacro)
@@ -7,5 +7,6 @@
   <xacro:property name="visual_mesh_file" value="file://$(find hydrone_aerial_underwater_description)/meshes/hydrone_base.dae"/>
   <!-- Mass, see p.28 in Berg2012 -->
-  <xacro:property name="mass" value="1.42887"/>
+  <!-- <xacro:property name="mass" value="1.93"/> -->
+  <xacro:property name="mass" value="1862.87"/>
   <xacro:property name="namespace" value="$(arg namespace)" />
   <xacro:property name="rotor_velocity_slowdown_sim" value="10" />
@@ -14,5 +15,4 @@
   <xacro:property name="rotor_1_mesh_file" value="package://hydrone_aerial_underwater_description/meshes/aerial_propeller_1.dae" />
   <xacro:property name="rotor_2_mesh_file" value="package://hydrone_aerial_underwater_description/meshes/aerial_propeller_2.dae" />
-  <xacro:property name="mass" value="1.5" /> <!-- [kg] -->
   <xacro:property name="body_width" value="0.47" /> <!-- [m] -->
   <xacro:property name="body_height" value="0.09" /> <!-- [m] -->
@@ -28,5 +28,5 @@
   <xacro:property name="time_constant_up" value="0.0125" /> <!-- [s] -->
   <xacro:property name="time_constant_down" value="0.025" /> <!-- [s] -->
-  <xacro:property name="max_rot_velocity" value="838" /> <!-- [rad/s] -->
+  <xacro:property name="max_rot_velocity" value="11111838" /> <!-- [rad/s] -->
   <xacro:property name="sin30" value="0.5" />
   <xacro:property name="cos30" value="0.866025403784" />
@@ -54,26 +54,11 @@
   <xacro:macro name="hydrone_aerial_underwater_base"
     params="namespace *gazebo use_simplified_mesh inertial_reference_frame">
-    <!-- <link name="${namespace}/base_link">
-      <inertial>
-        <mass value="${mass}"/>
-        <origin xyz="0 0 0.115" rpy="0 0 0"/>
-        <inertia ixx="0.0347563" ixy="0.0" ixz="0.0" iyy="0.0458929" iyz="0.0" izz="0.0977" />
-      </inertial>
-      <visual>
-          <origin xyz="-0.2175 0.2175 0.05" rpy="1.5707 0 0"/>
-          <geometry>
-            <mesh filename="${visual_mesh_file}" scale="1 1 1"/>
-          </geometry>
-      </visual>
-      <collision>
-        <origin xyz="-0.0 0.0 0.1" rpy="0 0 0"/>
-        <geometry>
-          <box size="0.44 0.44 0.05"/>
-        </geometry>
-      </collision>
-    </link> -->
     <!-- Property Blocks -->
     <xacro:property name="body_inertia">
-      <inertia ixx="0.0347563" ixy="0.0" ixz="0.0" iyy="0.0458929" iyz="0.0" izz="0.0977" />
+      <!-- Iris values -->
+      <!-- <inertia ixx="0.0347563" ixy="0.0" ixz="0.0" iyy="0.0458929" iyz="0.0" izz="0.0977" /> -->
+      <!-- RexRov Values -->
+      <inertia ixx="525.39" ixy="1.44" ixz="33.41" iyy="794.20" iyz="2.6" izz="691.23"/>
+      <!-- <inertia ixx="0.52539" ixy="0.00144" ixz="0.03341" iyy="0.79420" iyz="0.0026" izz="0.69123"/> -->
       <!-- <inertia ixx="0.01152" ixy="0.0" ixz="0.0" iyy="0.01152" iyz="0.0" izz="0.0218" /> -->
     </xacro:property>
@@ -116,12 +101,12 @@
       </visual>
       <collision>
-        <origin xyz="-0.03 -0.0315 -0.01" rpy="0 0 0"/>
-        <geometry>
+        <!--<origin xyz="-0.03 -0.0315 -0.01" rpy="0 0 0"/>
+         <geometry>
           <mesh filename="file://$(find hydrone_aerial_underwater_description)/meshes/aquatic_propeller_1.dae" scale="1 1 1"/>
-        </geometry>
-        <!-- <origin xyz="-0.0 -0.0 -0.0" rpy="0 0 0"/>
+        </geometry> -->
+        <origin xyz="0.0 0.0 0.0" rpy="0 0 0"/>
         <geometry>
           <box size="0.06 0.06 0.04"/>
-        </geometry> -->
+        </geometry>
       </collision>
     </link>
@@ -141,6 +126,6 @@
         <clampMin>3000</clampMin>
         <!-- Minimum and maximum thrust force output allowed -->
-        <thrustMin>-50</thrustMin>
-        <thrustMax>50</thrustMax>
+        <thrustMin>-1000</thrustMin>
+        <thrustMax>1000</thrustMax>
         <!--
         Value from 0 to 1 to set the efficiency of the output thrust force
@@ -161,5 +146,5 @@
         <conversion>
           <type>Basic</type>
-          <rotorConstant>0.0002</rotorConstant>
+          <rotorConstant>0.00031</rotorConstant>
         </conversion>
       </plugin>
@@ -180,12 +165,12 @@
       </xacro:box_inertial>
       <collision>
-        <origin xyz="-0.03 -0.0315 -0.01" rpy="0 0 0"/>
+        <!-- <origin xyz="-0.03 -0.0315 -0.01" rpy="0 0 0"/>
         <geometry>
           <mesh filename="file://$(find hydrone_aerial_underwater_description)/meshes/aquatic_propeller.dae" scale="1 1 1"/>
-        </geometry>
-        <!-- <origin xyz="-0.0 -0.0 -0.0" rpy="0 0 0"/>
+        </geometry> -->
+        <origin xyz="-0.0 -0.0 -0.0" rpy="0 0 0"/>
         <geometry>
           <box size="0.06 0.06 0.04"/>
-        </geometry> -->
+        </geometry>
       </collision>
       <visual>
@@ -211,6 +196,6 @@
         <clampMin>3000</clampMin>
         <!-- Minimum and maximum thrust force output allowed -->
-        <thrustMin>-50</thrustMin>
-        <thrustMax>50</thrustMax>
+        <thrustMin>-1000</thrustMin>
+        <thrustMax>1000</thrustMax>
         <!--
         Value from 0 to 1 to set the efficiency of the output thrust force
@@ -231,5 +216,5 @@
         <conversion>
           <type>Basic</type>
-          <rotorConstant>0.0002</rotorConstant>
+          <rotorConstant>0.00031</rotorConstant>
         </conversion>
       </plugin>
@@ -250,12 +235,12 @@
       </xacro:box_inertial>
       <collision>
-        <origin xyz="-0.03 -0.0315 -0.01" rpy="0 0 0"/>
+        <!-- <origin xyz="-0.03 -0.0315 -0.01" rpy="0 0 0"/>
         <geometry>
           <mesh filename="file://$(find hydrone_aerial_underwater_description)/meshes/aquatic_propeller_1.dae" scale="1 1 1"/>
-        </geometry>
-        <!-- <origin xyz="-0.0 -0.0 -0.0" rpy="0 0 0"/>
+        </geometry> -->
+        <origin xyz="-0.0 -0.0 -0.0" rpy="0 0 0"/>
         <geometry>
           <box size="0.06 0.06 0.04"/>
-        </geometry> -->
+        </geometry>
       </collision>
       <visual>
@@ -281,6 +266,6 @@
         <clampMin>3000</clampMin>
         <!-- Minimum and maximum thrust force output allowed -->
-        <thrustMin>-50</thrustMin>
-        <thrustMax>50</thrustMax>
+        <thrustMin>-1000</thrustMin>
+        <thrustMax>1000</thrustMax>
         <!--
         Value from 0 to 1 to set the efficiency of the output thrust force
@@ -301,5 +286,5 @@
         <conversion>
           <type>Basic</type>
-          <rotorConstant>0.0002</rotorConstant>
+          <rotorConstant>0.00031</rotorConstant>
         </conversion>
       </plugin>
@@ -320,12 +305,12 @@
       </xacro:box_inertial>
       <collision>
-        <origin xyz="-0.03 -0.0315 -0.01" rpy="0 0 0"/>
+        <!-- <origin xyz="-0.03 -0.0315 -0.01" rpy="0 0 0"/>
         <geometry>
           <mesh filename="file://$(find hydrone_aerial_underwater_description)/meshes/aquatic_propeller.dae" scale="1 1 1"/>
-        </geometry>
-        <!-- <origin xyz="-0.0 -0.0 -0.0" rpy="0 0 0"/>
+        </geometry> -->
+        <origin xyz="-0.0 -0.0 -0.0" rpy="0 0 0"/>
         <geometry>
           <box size="0.06 0.06 0.04"/>
-        </geometry> -->
+        </geometry>
       </collision>
       <visual>
@@ -351,6 +336,6 @@
         <clampMin>3000</clampMin>
         <!-- Minimum and maximum thrust force output allowed -->
-        <thrustMin>-50</thrustMin>
-        <thrustMax>50</thrustMax>
+        <thrustMin>-1000</thrustMin>
+        <thrustMax>1000</thrustMax>
         <!--
         Value from 0 to 1 to set the efficiency of the output thrust force
@@ -371,5 +356,5 @@
         <conversion>
           <type>Basic</type>
-          <rotorConstant>0.0002</rotorConstant>
+          <rotorConstant>0.00031</rotorConstant>
         </conversion>
       </plugin>
