Commit message: sdfds

File: hydrone_aerial_underwater_description/urdf/hydrone_aerial_underwater.gazebo.xacro (robot description, xacro)
@@ -6,8 +6,8 @@
     assume NWU (otherwise cob is below cog?).
     -->
-    <xacro:property name="cob" value="0.0 0.0 0.3"/>
+    <xacro:property name="cob" value="0.0 0.0 0.0"/>
     <!-- Volume, see p.31 in Berg2012 -->
-    <xacro:property name="volume" value="1.83826"/>
-    <!-- <xacro:property name="volume" value="0.00142887 "/> -->
+    <!-- <xacro:property name="volume" value="1.83826"/> -->
+    <xacro:property name="volume" value="0.0052887"/>
     <xacro:macro name="hydrone_aerial_underwater_hydro_model" params="namespace">
         <link name="${namespace}/base_link">
@@ -15,13 +15,37 @@
             <volume>${volume}</volume>
             <box>
-                <width>1.5</width>
-                <length>2.6</length>
-                <height>1.6</height>
+                <width>0.47</width>
+                <length>0.47</length>
+                <height>0.2</height>
             </box>
             <center_of_buoyancy>${cob}</center_of_buoyancy>
             <hydrodynamic_model>
                 <type>fossen</type>
+                <!-- <added_mass>
+                    1.93       0.0         0.0         0.0         0.0         0.0
+                    0.0         1.93       0.0         0.0         0.0         0.0
+                    0.0         0.0         1.93       0.0         0.0         0.0
+                    0.0         0.0         0.0         0.0156   0.0014   0.0004
+                    0.0         0.0         0.0         0.0014    0.03      0.0011
+                    0.0         0.0         0.0         0.0004    0.0011  0.0166
+                </added_mass>
+                <linear_damping>
+                    0.0125   0.0         0.0         0.0         0.0         0.0
+                    0.0         0.0125   0.0         0.0         0.0         0.0
+                    0.0         0.0         0.0499   0.0         0.0         0.0
+                    0.0         0.0         0.0         0.0125   0.0         0.0
+                    0.0         0.0         0.0         0.0         0.0125   0.0
+                    0.0         0.0         0.0         0.0         0.0         0.0499
+                </linear_damping>
+                <quadratic_damping>
+                    0.0125   0.0         0.0         0.0         0.0         0.0
+                    0.0         0.0125   0.0         0.0         0.0         0.0
+                    0.0         0.0         0.0499   0.0         0.0         0.0
+                    0.0         0.0         0.0         0.0125   0.0         0.0
+                    0.0         0.0         0.0         0.0         0.0125   0.0
+                    0.0         0.0         0.0         0.0         0.0         0.0499
+                </quadratic_damping>  -->
                 <!-- Added mass: see p.28 in Berg2012 -->
-                <added_mass>
+                <!-- <added_mass>
                      779.79 -6.8773 -103.32  8.5426 -165.54 -7.8033
                     -6.8773    1222   51.29  409.44 -5.8488  62.726
@@ -30,5 +54,5 @@
                     -165.54 -5.8488 -386.42 -10.027  842.69 -1.1162
                     -7.8033  62.726  10.775  21.019 -1.1162  224.32
-                </added_mass>
+                </added_mass> -->
                 <!-- <added_mass>
                      77.979 -0.68773 -10.332  0.85426 -16.554 -0.78033
@@ -39,5 +63,5 @@
                     -0.78033  6.2726  1.0775  2.1019 -0.11162  22.432
                 </added_mass> -->
-                <!-- <added_mass>
+                <added_mass>
                      0.77979 -0.0068773 -0.10332  0.00085426 -0.16554 -0.00078033
                     -0.0068773    1.222   0.05129  0.40944 -0.0058488  0.062726
@@ -46,19 +70,19 @@
                     -0.16554 -0.0058488 -0.38642 -0.010027  0.84269 -0.0011162
                     -0.078033  0.062726  0.010775  0.021019 -0.0011162  0.22432
-                </added_mass> -->
+                </added_mass>
                 <!-- Linear damping: see p.31 in Berg2012 -->
+                <!-- <linear_damping>
+                    -74.82 -69.48 -728.4 -268.8 -309.77 -105
+                </linear_damping> -->
                 <linear_damping>
-                    -74.82 -69.48 -728.4 -268.8 -309.77 -105
+                    -0.07482 -0.06948 -0.7284 -0.2688 -0.30977 -0.105
                 </linear_damping>
-                <!-- <linear_damping>
-                    -0.07482 -0.06948 -0.7284 -0.2688 -0.30977 -0.105
-                </linear_damping> -->
                 <!-- Non-linear damping: see p.30 in Berg2012 -->
+                <!-- <quadratic_damping>
+                    -748.22 -992.53 -1821.01 -672 -774.44 -523.27
+                </quadratic_damping> -->
                 <quadratic_damping>
-                    -748.22 -992.53 -1821.01 -672 -774.44 -523.27
+                    -0.74822 -0.99253 -1.82101 -0.672 -0.77444 -0.52327
                 </quadratic_damping>
-                <!-- <quadratic_damping>
-                    -0.74822 -0.99253 -1.82101 -0.672 -0.77444 -0.52327
-                </quadratic_damping> -->
             </hydrodynamic_model>
         </link>

File: hydrone_aerial_underwater_description/urdf/hydrone_aerial_underwater_base.xacro (robot description, xacro)
@@ -7,6 +7,6 @@
   <xacro:property name="visual_mesh_file" value="file://$(find hydrone_aerial_underwater_description)/meshes/hydrone_base.dae"/>
   <!-- Mass, see p.28 in Berg2012 -->
-  <!-- <xacro:property name="mass" value="1.93"/> -->
-  <xacro:property name="mass" value="1862.87"/>
+  <xacro:property name="mass" value="1.93"/>
+  <!-- <xacro:property name="mass" value="1862.87"/> -->
   <xacro:property name="namespace" value="$(arg namespace)" />
   <xacro:property name="rotor_velocity_slowdown_sim" value="10" />
@@ -57,7 +57,7 @@
     <xacro:property name="body_inertia">
       <!-- Iris values -->
-      <!-- <inertia ixx="0.0347563" ixy="0.0" ixz="0.0" iyy="0.0458929" iyz="0.0" izz="0.0977" /> -->
+      <inertia ixx="0.0347563" ixy="0.0" ixz="0.0" iyy="0.0458929" iyz="0.0" izz="0.0977" />
       <!-- RexRov Values -->
-      <inertia ixx="525.39" ixy="1.44" ixz="33.41" iyy="794.20" iyz="2.6" izz="691.23"/>
+      <!-- <inertia ixx="525.39" ixy="1.44" ixz="33.41" iyy="794.20" iyz="2.6" izz="691.23"/> -->
       <!-- <inertia ixx="0.52539" ixy="0.00144" ixz="0.03341" iyy="0.79420" iyz="0.0026" izz="0.69123"/> -->
       <!-- <inertia ixx="0.01152" ixy="0.0" ixz="0.0" iyy="0.01152" iyz="0.0" izz="0.0218" /> -->
@@ -88,10 +88,7 @@
     </joint>
     <link name="${namespace}/thruster_1">
-      <xacro:box_inertial x="0" y="0" z="0" mass="0.001">
+      <xacro:box_inertial x="0" y="0" z="0" mass="0.0001">
         <origin xyz="0 0 0" rpy="0 0 0"/>
       </xacro:box_inertial>
-      <!-- <xacro:box_inertial x="0.000088464" y="0.000092478" z="0.000152266" mass="0.011">
-        <origin xyz="0 0 0" rpy="0 0 0"/>
-      </xacro:box_inertial> -->
       <visual>
         <origin xyz="-0.03 -0.0315 -0.01" rpy="0 0 0"/>
@@ -101,8 +98,4 @@
       </visual>
       <collision>
-        <!--<origin xyz="-0.03 -0.0315 -0.01" rpy="0 0 0"/>
-         <geometry>
-          <mesh filename="file://$(find hydrone_aerial_underwater_description)/meshes/aquatic_propeller_1.dae" scale="1 1 1"/>
-        </geometry> -->
         <origin xyz="0.0 0.0 0.0" rpy="0 0 0"/>
         <geometry>
@@ -113,30 +106,13 @@
     <gazebo>
       <plugin name="${namespace}_0_thruster_model" filename="libuuv_thruster_ros_plugin.so">
-        <!-- Name of the thruster link -->
         <linkName>${namespace}/thruster_1</linkName>
-        <!-- Name of the joint between thruster and vehicle base link -->
         <jointName>${namespace}/thruster_1_joint</jointName>
-        <!-- Make the thruster aware of its id -->
         <thrusterID>1</thrusterID>
-        <!-- Gain of the input command signal -->
         <gain>1</gain>
-        <!-- Maximum allowed input value for the input signal for thruster unit -->
         <clampMax>-3000</clampMax>
-        <!-- Minimum allowed value for the input signal for thruster unit -->
         <clampMin>3000</clampMin>
-        <!-- Minimum and maximum thrust force output allowed -->
         <thrustMin>-1000</thrustMin>
         <thrustMax>1000</thrustMax>
-        <!--
-        Value from 0 to 1 to set the efficiency of the output thrust force
-        Default value is 1.0
-        -->
         <thrust_efficiency>1</thrust_efficiency>
-        <!--
-        Value from 0 to 1 to set the efficiency of the propeller as a factor
-        to be multiplied to the current value of the state variable at each
-        iteration.
-        Default value is 1.0
-        -->
         <propeller_efficiency>1</propeller_efficiency>
         <dynamics>
@@ -161,12 +137,8 @@
     </joint>
     <link name="${namespace}/thruster_2">
-      <xacro:box_inertial x="0" y="0" z="0" mass="0.001">
+      <xacro:box_inertial x="0" y="0" z="0" mass="0.0001">
         <origin xyz="0 0 0" rpy="0 0 0"/>
       </xacro:box_inertial>
       <collision>
-        <!-- <origin xyz="-0.03 -0.0315 -0.01" rpy="0 0 0"/>
-        <geometry>
-          <mesh filename="file://$(find hydrone_aerial_underwater_description)/meshes/aquatic_propeller.dae" scale="1 1 1"/>
-        </geometry> -->
         <origin xyz="-0.0 -0.0 -0.0" rpy="0 0 0"/>
         <geometry>
@@ -183,30 +155,13 @@
     <gazebo>
       <plugin name="${namespace}_2_thruster_model" filename="libuuv_thruster_ros_plugin.so">
-        <!-- Name of the thruster link -->
         <linkName>${namespace}/thruster_2</linkName>
-        <!-- Name of the joint between thruster and vehicle base link -->
         <jointName>${namespace}/thruster_2_joint</jointName>
-        <!-- Make the thruster aware of its id -->
         <thrusterID>2</thrusterID>
-        <!-- Gain of the input command signal -->
         <gain>1</gain>
-        <!-- Maximum allowed input value for the input signal for thruster unit -->
         <clampMax>-3000</clampMax>
-        <!-- Minimum allowed value for the input signal for thruster unit -->
         <clampMin>3000</clampMin>
-        <!-- Minimum and maximum thrust force output allowed -->
         <thrustMin>-1000</thrustMin>
         <thrustMax>1000</thrustMax>
-        <!--
-        Value from 0 to 1 to set the efficiency of the output thrust force
-        Default value is 1.0
-        -->
         <thrust_efficiency>1</thrust_efficiency>
-        <!--
-        Value from 0 to 1 to set the efficiency of the propeller as a factor
-        to be multiplied to the current value of the state variable at each
-        iteration.
-        Default value is 1.0
-        -->
         <propeller_efficiency>1</propeller_efficiency>
         <dynamics>
@@ -231,12 +186,8 @@
     </joint>
     <link name="${namespace}/thruster_3">
-      <xacro:box_inertial x="0" y="0" z="0" mass="0.001">
+      <xacro:box_inertial x="0" y="0" z="0" mass="0.0001">
         <origin xyz="0 0 0" rpy="0 0 0"/>
       </xacro:box_inertial>
       <collision>
-        <!-- <origin xyz="-0.03 -0.0315 -0.01" rpy="0 0 0"/>
-        <geometry>
-          <mesh filename="file://$(find hydrone_aerial_underwater_description)/meshes/aquatic_propeller_1.dae" scale="1 1 1"/>
-        </geometry> -->
         <origin xyz="-0.0 -0.0 -0.0" rpy="0 0 0"/>
         <geometry>
@@ -253,30 +204,13 @@
     <gazebo>
       <plugin name="${namespace}_3_thruster_model" filename="libuuv_thruster_ros_plugin.so">
-        <!-- Name of the thruster link -->
         <linkName>${namespace}/thruster_3</linkName>
-        <!-- Name of the joint between thruster and vehicle base link -->
         <jointName>${namespace}/thruster_3_joint</jointName>
-        <!-- Make the thruster aware of its id -->
         <thrusterID>3</thrusterID>
-        <!-- Gain of the input command signal -->
         <gain>1</gain>
-        <!-- Maximum allowed input value for the input signal for thruster unit -->
         <clampMax>-3000</clampMax>
-        <!-- Minimum allowed value for the input signal for thruster unit -->
         <clampMin>3000</clampMin>
-        <!-- Minimum and maximum thrust force output allowed -->
         <thrustMin>-1000</thrustMin>
         <thrustMax>1000</thrustMax>
-        <!--
-        Value from 0 to 1 to set the efficiency of the output thrust force
-        Default value is 1.0
-        -->
         <thrust_efficiency>1</thrust_efficiency>
-        <!--
-        Value from 0 to 1 to set the efficiency of the propeller as a factor
-        to be multiplied to the current value of the state variable at each
-        iteration.
-        Default value is 1.0
-        -->
         <propeller_efficiency>1</propeller_efficiency>
         <dynamics>
@@ -301,12 +235,8 @@
     </joint>
     <link name="${namespace}/thruster_4">
-      <xacro:box_inertial x="0" y="0" z="0" mass="0.001">
+      <xacro:box_inertial x="0" y="0" z="0" mass="0.0001">
         <origin xyz="0 0 0" rpy="0 0 0"/>
       </xacro:box_inertial>
       <collision>
-        <!-- <origin xyz="-0.03 -0.0315 -0.01" rpy="0 0 0"/>
-        <geometry>
-          <mesh filename="file://$(find hydrone_aerial_underwater_description)/meshes/aquatic_propeller.dae" scale="1 1 1"/>
-        </geometry> -->
         <origin xyz="-0.0 -0.0 -0.0" rpy="0 0 0"/>
         <geometry>
@@ -323,30 +253,13 @@
     <gazebo>
       <plugin name="${namespace}_4_thruster_model" filename="libuuv_thruster_ros_plugin.so">
-        <!-- Name of the thruster link -->
         <linkName>${namespace}/thruster_4</linkName>
-        <!-- Name of the joint between thruster and vehicle base link -->
         <jointName>${namespace}/thruster_4_joint</jointName>
-        <!-- Make the thruster aware of its id -->
         <thrusterID>4</thrusterID>
-        <!-- Gain of the input command signal -->
         <gain>1</gain>
-        <!-- Maximum allowed input value for the input signal for thruster unit -->
         <clampMax>-3000</clampMax>
-        <!-- Minimum allowed value for the input signal for thruster unit -->
         <clampMin>3000</clampMin>
-        <!-- Minimum and maximum thrust force output allowed -->
         <thrustMin>-1000</thrustMin>
         <thrustMax>1000</thrustMax>
-        <!--
-        Value from 0 to 1 to set the efficiency of the output thrust force
-        Default value is 1.0
-        -->
         <thrust_efficiency>1</thrust_efficiency>
-        <!--
-        Value from 0 to 1 to set the efficiency of the propeller as a factor
-        to be multiplied to the current value of the state variable at each
-        iteration.
-        Default value is 1.0
-        -->
         <propeller_efficiency>1</propeller_efficiency>
         <dynamics>

Commit message: 0_o

File: hydrone_aerial_underwater_description/urdf/hydrone_aerial_underwater.gazebo.xacro (robot description, xacro)
@@ -9,5 +9,5 @@
     <!-- Volume, see p.31 in Berg2012 -->
     <!-- <xacro:property name="volume" value="1.83826"/> -->
-    <xacro:property name="volume" value="0.0052887"/>
+    <xacro:property name="volume" value="0.0022887"/>
     <xacro:macro name="hydrone_aerial_underwater_hydro_model" params="namespace">
         <link name="${namespace}/base_link">
@@ -22,5 +22,5 @@
             <hydrodynamic_model>
                 <type>fossen</type>
-                <!-- <added_mass>
+                <added_mass>
                     1.93       0.0         0.0         0.0         0.0         0.0
                     0.0         1.93       0.0         0.0         0.0         0.0
@@ -38,5 +38,5 @@
                     0.0         0.0         0.0         0.0         0.0         0.0499
                 </linear_damping>
-                <quadratic_damping>
+                <!-- <quadratic_damping>
                     0.0125   0.0         0.0         0.0         0.0         0.0
                     0.0         0.0125   0.0         0.0         0.0         0.0
@@ -63,5 +63,5 @@
                     -0.78033  6.2726  1.0775  2.1019 -0.11162  22.432
                 </added_mass> -->
-                <added_mass>
+                <!-- <added_mass>
                      0.77979 -0.0068773 -0.10332  0.00085426 -0.16554 -0.00078033
                     -0.0068773    1.222   0.05129  0.40944 -0.0058488  0.062726
@@ -70,12 +70,12 @@
                     -0.16554 -0.0058488 -0.38642 -0.010027  0.84269 -0.0011162
                     -0.078033  0.062726  0.010775  0.021019 -0.0011162  0.22432
-                </added_mass>
+                </added_mass> -->
                 <!-- Linear damping: see p.31 in Berg2012 -->
                 <!-- <linear_damping>
                     -74.82 -69.48 -728.4 -268.8 -309.77 -105
                 </linear_damping> -->
-                <linear_damping>
+                <!-- <linear_damping>
                     -0.07482 -0.06948 -0.7284 -0.2688 -0.30977 -0.105
-                </linear_damping>
+                </linear_damping> -->
                 <!-- Non-linear damping: see p.30 in Berg2012 -->
                 <!-- <quadratic_damping>

File: hydrone_aerial_underwater_description/urdf/hydrone_aerial_underwater_base.xacro (robot description, xacro)
@@ -81,5 +81,5 @@
       <xacro:insert_block name="body_inertia" />
     </xacro:multirotor_base_macro>
-    <joint name="${namespace}/thruster_1_joint" type="continuous">
+    <!-- <joint name="${namespace}/thruster_1_joint" type="continuous">
       <origin xyz="0.19725 -0.19725 -0.055" rpy="0 0 0"/>
       <axis xyz="0 0 1"/>
@@ -88,5 +88,5 @@
     </joint>
     <link name="${namespace}/thruster_1">
-      <xacro:box_inertial x="0" y="0" z="0" mass="0.0001">
+      <xacro:box_inertial x="0" y="0" z="0" mass="0.1">
         <origin xyz="0 0 0" rpy="0 0 0"/>
       </xacro:box_inertial>
@@ -137,5 +137,5 @@
     </joint>
     <link name="${namespace}/thruster_2">
-      <xacro:box_inertial x="0" y="0" z="0" mass="0.0001">
+      <xacro:box_inertial x="0" y="0" z="0" mass="0.1">
         <origin xyz="0 0 0" rpy="0 0 0"/>
       </xacro:box_inertial>
@@ -186,5 +186,5 @@
     </joint>
     <link name="${namespace}/thruster_3">
-      <xacro:box_inertial x="0" y="0" z="0" mass="0.0001">
+      <xacro:box_inertial x="0" y="0" z="0" mass="0.1">
         <origin xyz="0 0 0" rpy="0 0 0"/>
       </xacro:box_inertial>
@@ -235,5 +235,5 @@
     </joint>
     <link name="${namespace}/thruster_4">
-      <xacro:box_inertial x="0" y="0" z="0" mass="0.0001">
+      <xacro:box_inertial x="0" y="0" z="0" mass="0.1">
         <origin xyz="0 0 0" rpy="0 0 0"/>
       </xacro:box_inertial>
@@ -276,5 +276,5 @@
       <selfCollide>false</selfCollide>
       <material>Gazebo/Blue</material>
-    </gazebo>
+    </gazebo> -->
     <gazebo reference="${namespace}/base_link">
       <material>Gazebo/White</material>

File: hydrone_aerial_underwater_description/urdf/multirotor_base.xacro (robot description, xacro)
@@ -132,4 +132,26 @@
       </plugin>
     </gazebo>
+    <gazebo>
+      <plugin name="${namespace}_4_thruster_model" filename="libuuv_thruster_ros_plugin.so">
+        <linkName>${robot_namespace}/rotor_${motor_number}</linkName>
+        <jointName>${robot_namespace}/rotor_${motor_number}_joint</jointName>
+        <thrusterID>${motor_number}</thrusterID>
+        <gain>1</gain>
+        <clampMax>-3000</clampMax>
+        <clampMin>3000</clampMin>
+        <thrustMin>-1000</thrustMin>
+        <thrustMax>1000</thrustMax>
+        <thrust_efficiency>1</thrust_efficiency>
+        <propeller_efficiency>1</propeller_efficiency>
+        <dynamics>
+          <type>FirstOrder</type>
+          <timeConstant>0.05</timeConstant>
+        </dynamics>
+        <conversion>
+          <type>Basic</type>
+          <rotorConstant>0.00031</rotorConstant>
+        </conversion>
+      </plugin>
+    </gazebo>
     <gazebo reference="${robot_namespace}/rotor_${motor_number}">
       <material>Gazebo/${color}</material>

Commit message: asdf

File: hydrone_aerial_underwater_description/urdf/hydrone_aerial_underwater.gazebo.xacro (robot description, xacro)
@@ -9,5 +9,5 @@
     <!-- Volume, see p.31 in Berg2012 -->
     <!-- <xacro:property name="volume" value="1.83826"/> -->
-    <xacro:property name="volume" value="0.0022887"/>
+    <xacro:property name="volume" value="0.0010887"/>
     <xacro:macro name="hydrone_aerial_underwater_hydro_model" params="namespace">
         <link name="${namespace}/base_link">

File: hydrone_aerial_underwater_description/urdf/hydrone_aerial_underwater_base.xacro (robot description, xacro)
@@ -17,5 +17,4 @@
   <xacro:property name="body_width" value="0.47" /> <!-- [m] -->
   <xacro:property name="body_height" value="0.09" /> <!-- [m] -->
-  <xacro:property name="mass_rotor" value="0.005" /> <!-- [kg] -->
   <xacro:property name="arm_length_front_x" value="0.19725" /> <!-- [m] -->
   <xacro:property name="arm_length_back_x" value="0.19725" /> <!-- [m] -->
@@ -24,14 +23,15 @@
   <xacro:property name="rotor_offset_top" value="0.035" /> <!-- [m] -->
   <xacro:property name="radius_rotor" value="0.195" /> <!-- [m] -->
+  <xacro:property name="sin30" value="0.5" />
+  <xacro:property name="cos30" value="0.866025403784" />
+  <xacro:property name="sqrt2" value="1.4142135623730951" />
+  <xacro:property name="mass_rotor" value="0.005" /> <!-- [kg] -->
+  <xacro:property name="rotor_drag_coefficient" value="8.06428e-05" />
+  <xacro:property name="rolling_moment_coefficient" value="0.000001" />
   <xacro:property name="motor_constant" value="8.54858e-06" /> <!-- [kg.m/s^2] -->
   <xacro:property name="moment_constant" value="0.016" /> <!-- [m] -->
   <xacro:property name="time_constant_up" value="0.0125" /> <!-- [s] -->
   <xacro:property name="time_constant_down" value="0.025" /> <!-- [s] -->
-  <xacro:property name="max_rot_velocity" value="11111838" /> <!-- [rad/s] -->
-  <xacro:property name="sin30" value="0.5" />
-  <xacro:property name="cos30" value="0.866025403784" />
-  <xacro:property name="sqrt2" value="1.4142135623730951" />
-  <xacro:property name="rotor_drag_coefficient" value="8.06428e-05" />
-  <xacro:property name="rolling_moment_coefficient" value="0.000001" />
+  <xacro:property name="max_rot_velocity" value="838" /> <!-- [rad/s] -->
   <xacro:property name="mesh_pos_x" value="-0.2175" /> <!-- [m] -->
   <xacro:property name="mesh_pos_y" value="0.2175" /> <!-- [m] -->
