Commit message: 0_o

File: hydrone_aerial_underwater_description/urdf/hydrone_aerial_underwater.gazebo.xacro (robot description, xacro)
@@ -9,5 +9,5 @@
     <!-- Volume, see p.31 in Berg2012 -->
     <!-- <xacro:property name="volume" value="1.83826"/> -->
-    <xacro:property name="volume" value="0.0010887"/>
+    <xacro:property name="volume" value="0.0016"/>
     <xacro:macro name="hydrone_aerial_underwater_hydro_model" params="namespace">
         <link name="${namespace}/base_link">
@@ -17,5 +17,5 @@
                 <width>0.47</width>
                 <length>0.47</length>
-                <height>0.2</height>
+                <height>0.1</height>
             </box>
             <center_of_buoyancy>${cob}</center_of_buoyancy>

Commit message: 0_x

File: hydrone_aerial_underwater_description/urdf/hydrone_aerial_underwater.gazebo.xacro (robot description, xacro)
@@ -9,5 +9,6 @@
     <!-- Volume, see p.31 in Berg2012 -->
     <!-- <xacro:property name="volume" value="1.83826"/> -->
-    <xacro:property name="volume" value="0.0016"/>
+    <!-- <xacro:property name="volume" value="0.00001"/> -->
+    <xacro:property name="volume" value="0.001"/>
     <xacro:macro name="hydrone_aerial_underwater_hydro_model" params="namespace">
         <link name="${namespace}/base_link">
@@ -88,4 +89,36 @@
         </link>
     </xacro:macro>
+    <gazebo reference="base_scan">
+        <material>Gazebo/FlatBlack</material>
+        <sensor type="ray" name="lds_lfcd_sensor">
+        <pose>0 0 0 0 0 0</pose>
+        <visualize>true</visualize>
+        <update_rate>5</update_rate>
+        <ray>
+            <scan>
+            <horizontal>
+                <samples>10</samples>
+                <resolution>1</resolution>
+                <min_angle>0.0</min_angle>
+                <max_angle>6.28319</max_angle>
+            </horizontal>
+            </scan>
+            <range>
+            <min>0.50</min>
+            <max>20.0</max>
+            <resolution>0.015</resolution>
+            </range>
+            <noise>
+            <type>gaussian</type>
+            <mean>0.0</mean>
+            <stddev>0.01</stddev>
+            </noise>
+        </ray>
+        <plugin name="gazebo_ros_lds_lfcd_controller" filename="libgazebo_ros_laser.so">
+            <topicName>scan</topicName>
+            <frameName>base_scan</frameName>
+        </plugin>
+        </sensor>
+    </gazebo>
 </robot>
 <!-- <added_mass>

File: hydrone_aerial_underwater_description/urdf/hydrone_aerial_underwater_base.xacro (robot description, xacro)
@@ -33,5 +33,5 @@
   <xacro:property name="time_constant_up" value="0.0125" /> <!-- [s] -->
   <xacro:property name="time_constant_down" value="0.025" /> <!-- [s] -->
-  <xacro:property name="max_rot_velocity" value="838" /> <!-- [rad/s] -->
+  <xacro:property name="max_rot_velocity" value="1838" /> <!-- [rad/s] -->
   <xacro:property name="mesh_pos_x" value="-0.2175" /> <!-- [m] -->
   <xacro:property name="mesh_pos_y" value="0.2175" /> <!-- [m] -->
@@ -50,4 +50,6 @@
     <xacro:box_inertia x="${radius_rotor}" y="0.015" z="0.003" mass="${mass_rotor*rotor_velocity_slowdown_sim}" />
   </xacro:property>
+  <xacro:arg name="gpu" default="false"/>
+  <xacro:property name="gpu" value="$(arg gpu)" />
   <!-- Included URDF Files -->
   <xacro:include filename="$(find hydrone_aerial_underwater_description)/urdf/multirotor_base.xacro" />
@@ -430,3 +432,34 @@
     <!-- <xacro:include filename="$(find hydrone_aerial_underwater_description)/urdf/hydrone_aerial_underwater_actuators.xacro" /> -->
   </xacro:macro>
+  <joint name="scan_joint" type="fixed">
+    <parent link="${namespace}/base_link"/>
+    <child link="base_scan"/>
+    <origin xyz="0.0 0 0.07" rpy="0 0 0"/>
+  </joint>
+  <link name="base_scan">
+    <visual>
+      <origin xyz="0 0 0.0" rpy="0 0 0"/>
+      <geometry>
+        <mesh filename="package://rexrov_ddpg/meshes/lds.stl" scale="0.001 0.001 0.001"/>
+      </geometry>
+      <material name="dark"/>
+    </visual>
+    <collision>
+      <origin xyz="0.015 0 -0.0065" rpy="0 0 0"/>
+      <geometry>
+        <cylinder length="0.0315" radius="0.055"/>
+      </geometry>
+    </collision>
+    <inertial>
+      <mass value="0.114" />
+      <origin xyz="0 0 0" />
+      <inertia ixx="0.001" ixy="0.0" ixz="0.0"
+              iyy="0.001" iyz="0.0"
+              izz="0.001" />
+    </inertial>
+  </link>
+  <!-- <xacro:include filename="$(find hydrone_aerial_underwater_description)/urdf/VLP-16.urdf.xacro"/>
+  <VLP-16 parent="${namespace}/base_link" name="velodyne" topic="/velodyne_points" hz="10" samples="440" gpu="${gpu}">
+    <origin xyz="0 0 0.05" rpy="0 0 0" />
+  </VLP-16> -->
 </robot>

Commit message: 0_o

File: hydrone_aerial_underwater_description/urdf/hydrone_aerial_underwater.gazebo.xacro (robot description, xacro)
@@ -100,6 +100,6 @@
                 <samples>10</samples>
                 <resolution>1</resolution>
-                <min_angle>0.0</min_angle>
-                <max_angle>6.28319</max_angle>
+                <min_angle>-1.570796</min_angle>
+                <max_angle>1.570796</max_angle>
             </horizontal>
             </scan>
@@ -121,4 +121,27 @@
         </sensor>
     </gazebo>
+     <!-- <gazebo reference="base_scan">
+        <sensor:ray name="laser">
+            <rayCount>180</rayCount>
+            <rangeCount>180</rangeCount>
+            <laserCount>1</laserCount>
+            <origin>0.0 0.0 0.0</origin>
+            <displayRays>false</displayRays>
+            <minAngle>-130</minAngle>
+            <maxAngle>130</maxAngle>
+            <minRange>0.08</minRange>
+            <maxRange>10.0</maxRange>
+            <resRange>0.01</resRange>
+            <updateRate>20</updateRate>
+            <controller:gazebo_ros_laser name="gazebo_ros_laser_controller" plugin="libgazebo_ros_laser.so">
+            <gaussianNoise>0.005</gaussianNoise>
+            <alwaysOn>true</alwaysOn>
+            <updateRate>20</updateRate>
+            <topicName>scan</topicName>
+            <frameName>laser</frameName>
+            <interface:laser name="gazebo_ros_laser_iface" />
+            </controller:gazebo_ros_laser>
+        </sensor:ray>
+    </gazebo>  -->
 </robot>
 <!-- <added_mass>

Commit message: asdfasd

File: hydrone_aerial_underwater_description/urdf/hydrone_aerial_underwater.gazebo.xacro (robot description, xacro)
@@ -121,27 +121,36 @@
         </sensor>
     </gazebo>
-     <!-- <gazebo reference="base_scan">
-        <sensor:ray name="laser">
-            <rayCount>180</rayCount>
-            <rangeCount>180</rangeCount>
-            <laserCount>1</laserCount>
-            <origin>0.0 0.0 0.0</origin>
-            <displayRays>false</displayRays>
-            <minAngle>-130</minAngle>
-            <maxAngle>130</maxAngle>
-            <minRange>0.08</minRange>
-            <maxRange>10.0</maxRange>
-            <resRange>0.01</resRange>
-            <updateRate>20</updateRate>
-            <controller:gazebo_ros_laser name="gazebo_ros_laser_controller" plugin="libgazebo_ros_laser.so">
-            <gaussianNoise>0.005</gaussianNoise>
-            <alwaysOn>true</alwaysOn>
-            <updateRate>20</updateRate>
+    <!-- <gazebo reference="base_scan">
+        <material>Gazebo/FlatBlack</material>
+        <sensor type="ray" name="lds_lfcd_sensor">
+        <pose>0 0 0 0 0 0</pose>
+        <visualize>true</visualize>
+        <update_rate>5</update_rate>
+        <ray>
+            <scan>
+            <horizontal>
+                <samples>10</samples>
+                <resolution>1</resolution>
+                <min_angle>-0.78539816339</min_angle>
+                <max_angle>0.78539816339</max_angle>
+            </horizontal>
+            </scan>
+            <range>
+            <min>0.50</min>
+            <max>20.0</max>
+            <resolution>0.015</resolution>
+            </range>
+            <noise>
+            <type>gaussian</type>
+            <mean>0.0</mean>
+            <stddev>0.01</stddev>
+            </noise>
+        </ray>
+        <plugin name="gazebo_ros_lds_lfcd_controller" filename="libgazebo_ros_laser.so">
             <topicName>scan</topicName>
-            <frameName>laser</frameName>
-            <interface:laser name="gazebo_ros_laser_iface" />
-            </controller:gazebo_ros_laser>
-        </sensor:ray>
-    </gazebo>  -->
+            <frameName>base_scan</frameName>
+        </plugin>
+        </sensor>
+    </gazebo> -->
 </robot>
 <!-- <added_mass>
