Commit message: last

File: hydrone_aerial_underwater_description/urdf/VLP-16.urdf.xacro (robot description, xacro)
@@ -18,10 +18,10 @@
       <visual>
         <geometry>
-          <mesh filename="package://velodyne_description/meshes/VLP16_base_1.dae" />
+          <mesh filename="package://hydrone_aerial_underwater_description/meshes/VLP16_base_1.dae" />
         </geometry>
       </visual>
       <visual>
         <geometry>
-          <mesh filename="package://velodyne_description/meshes/VLP16_base_2.dae" />
+          <mesh filename="package://hydrone_aerial_underwater_description/meshes/VLP16_base_2.dae" />
         </geometry>
       </visual>
@@ -47,5 +47,5 @@
         <origin xyz="0 0 -0.0377" />
         <geometry>
-          <mesh filename="package://velodyne_description/meshes/VLP16_scan.dae" />
+          <mesh filename="package://hydrone_aerial_underwater_description/meshes/VLP16_scan.dae" />
         </geometry>
       </visual>

File: hydrone_aerial_underwater_description/urdf/hydrone_aerial_underwater.gazebo.xacro (robot description, xacro)
@@ -11,4 +11,5 @@
     <!-- <xacro:property name="volume" value="0.00001"/> -->
     <xacro:property name="volume" value="0.001"/>
+    <xacro:property name="M_PI" value="3.1415926535897931" />
     <xacro:macro name="hydrone_aerial_underwater_hydro_model" params="namespace">
         <link name="${namespace}/base_link">
@@ -39,5 +40,5 @@
                     0.0         0.0         0.0         0.0         0.0         0.0499
                 </linear_damping>
-                <!-- <quadratic_damping>
+                <quadratic_damping>
                     0.0125   0.0         0.0         0.0         0.0         0.0
                     0.0         0.0125   0.0         0.0         0.0         0.0
@@ -46,5 +47,5 @@
                     0.0         0.0         0.0         0.0         0.0125   0.0
                     0.0         0.0         0.0         0.0         0.0         0.0499
-                </quadratic_damping>  -->
+                </quadratic_damping>
                 <!-- Added mass: see p.28 in Berg2012 -->
                 <!-- <added_mass>
@@ -83,13 +84,13 @@
                     -748.22 -992.53 -1821.01 -672 -774.44 -523.27
                 </quadratic_damping> -->
-                <quadratic_damping>
+                <!-- <quadratic_damping>
                     -0.74822 -0.99253 -1.82101 -0.672 -0.77444 -0.52327
-                </quadratic_damping>
+                </quadratic_damping> -->
             </hydrodynamic_model>
         </link>
     </xacro:macro>
-    <gazebo reference="base_scan">
+    <!-- <gazebo reference="base_scan">
         <material>Gazebo/FlatBlack</material>
-        <sensor type="ray" name="lds_lfcd_sensor">
+        <sensor type="ray" name="VLP-16-VLP16-Simplified">
         <pose>0 0 0 0 0 0</pose>
         <visualize>true</visualize>
@@ -97,14 +98,22 @@
         <ray>
             <scan>
-            <horizontal>
-                <samples>20</samples>
-                <resolution>1</resolution>
-                <min_angle>-2.356194490192345</min_angle>
-                <max_angle>2.356194490192345</max_angle>
-            </horizontal>
+                <horizontal>
+                    <samples>8</samples>
+                    <resolution>1</resolution>
+                    <min_angle>-${3*M_PI/4}</min_angle>
+                    <max_angle>${3*M_PI/4}</max_angle>
+                    <min_angle>0</min_angle>
+                    <max_angle>${2*M_PI - M_PI/4}</max_angle>
+                </horizontal>
+                <vertical>
+                    <samples>5</samples>
+                    <resolution>1</resolution>
+                    <min_angle>-${15.0*M_PI/180.0}</min_angle>
+                    <max_angle>${15.0*M_PI/180.0}</max_angle>
+                </vertical>
             </scan>
             <range>
             <min>0.50</min>
-            <max>20.0</max>
+            <max>130.0</max>
             <resolution>0.015</resolution>
             </range>
@@ -112,5 +121,5 @@
             <type>gaussian</type>
             <mean>0.0</mean>
-            <stddev>0.01</stddev>
+            <stddev>0.0</stddev>
             </noise>
         </ray>
@@ -120,29 +129,29 @@
         </plugin>
         </sensor>
-    </gazebo>
-    <!-- <gazebo reference="base_scan">
+    </gazebo> -->
+    <gazebo reference="base_scan">
         <material>Gazebo/FlatBlack</material>
-        <sensor type="ray" name="lds_lfcd_sensor">
+        <sensor type="ray" name="Terafinder">
         <pose>0 0 0 0 0 0</pose>
         <visualize>true</visualize>
-        <update_rate>5</update_rate>
+        <update_rate>15</update_rate>
         <ray>
             <scan>
-            <horizontal>
-                <samples>10</samples>
-                <resolution>1</resolution>
-                <min_angle>-0.78539816339</min_angle>
-                <max_angle>0.78539816339</max_angle>
-            </horizontal>
+                <horizontal>
+                    <samples>8</samples>
+                    <resolution>1</resolution>
+                    <min_angle>0</min_angle>
+                    <max_angle>${2*M_PI - M_PI/4}</max_angle>
+                </horizontal>
             </scan>
             <range>
-            <min>0.50</min>
-            <max>20.0</max>
-            <resolution>0.015</resolution>
+            <min>0.5</min>
+            <max>7.5</max>
+            <resolution>0.01</resolution>
             </range>
             <noise>
             <type>gaussian</type>
             <mean>0.0</mean>
-            <stddev>0.01</stddev>
+            <stddev>0.0</stddev>
             </noise>
         </ray>
@@ -152,28 +161,300 @@
         </plugin>
         </sensor>
+    </gazebo>
+    <!-- <gazebo reference="base_ir_front_0">
+        <sensor type="ray" name="TeraRanger">
+            <pose>0 0 0 0 0 0</pose>
+            <visualize>true</visualize>
+            <update_rate>15</update_rate>
+            <ray>
+                <scan>
+                    <horizontal>
+                    <samples>10</samples>
+                    <resolution>1</resolution>
+                    <min_angle>-0.14835</min_angle>
+                    <max_angle>0.14835</max_angle>
+                    </horizontal>
+                    <vertical>
+                    <samples>10</samples>
+                    <resolution>1</resolution>
+                    <min_angle>-0.14835</min_angle>
+                    <max_angle>0.14835</max_angle>
+                    </vertical>
+                </scan>
+                <range>
+                    <min>0.01</min>
+                    <max>7.5</max>
+                    <resolution>0.01</resolution>
+                </range>
+            </ray>
+            <plugin filename="libgazebo_ros_range.so" name="gazebo_ros_range">
+                <gaussianNoise>0.005</gaussianNoise>
+                <alwaysOn>true</alwaysOn>
+                <updateRate>50</updateRate>
+                <topicName>sensor/ir_front_0</topicName>
+                <frameName>base_ir_front_0</frameName>
+                <radiation>INFRARED</radiation>
+                <fov>0.174533</fov>
+            </plugin>
+        </sensor>
+    </gazebo>
+    <gazebo reference="base_ir_front_45">
+        <sensor type="ray" name="TeraRanger">
+            <pose>0 0 0 0 0 0</pose>
+            <visualize>true</visualize>
+            <update_rate>15</update_rate>
+            <ray>
+                <scan>
+                    <horizontal>
+                    <samples>10</samples>
+                    <resolution>1</resolution>
+                    <min_angle>-0.14835</min_angle>
+                    <max_angle>0.14835</max_angle>
+                    </horizontal>
+                    <vertical>
+                    <samples>10</samples>
+                    <resolution>1</resolution>
+                    <min_angle>-0.14835</min_angle>
+                    <max_angle>0.14835</max_angle>
+                    </vertical>
+                </scan>
+                <range>
+                    <min>0.01</min>
+                    <max>7.5</max>
+                    <resolution>0.01</resolution>
+                </range>
+            </ray>
+            <plugin filename="libgazebo_ros_range.so" name="gazebo_ros_range">
+                <gaussianNoise>0.005</gaussianNoise>
+                <alwaysOn>true</alwaysOn>
+                <updateRate>50</updateRate>
+                <topicName>sensor/ir_front_45</topicName>
+                <frameName>base_ir_front_45</frameName>
+                <radiation>INFRARED</radiation>
+                <fov>0.174533</fov>
+            </plugin>
+        </sensor>
+    </gazebo>
+    <gazebo reference="base_ir_front_90">
+        <sensor type="ray" name="TeraRanger">
+            <pose>0 0 0 0 0 0</pose>
+            <visualize>true</visualize>
+            <update_rate>15</update_rate>
+            <ray>
+                <scan>
+                    <horizontal>
+                    <samples>10</samples>
+                    <resolution>1</resolution>
+                    <min_angle>-0.14835</min_angle>
+                    <max_angle>0.14835</max_angle>
+                    </horizontal>
+                    <vertical>
+                    <samples>10</samples>
+                    <resolution>1</resolution>
+                    <min_angle>-0.14835</min_angle>
+                    <max_angle>0.14835</max_angle>
+                    </vertical>
+                </scan>
+                <range>
+                    <min>0.01</min>
+                    <max>7.5</max>
+                    <resolution>0.01</resolution>
+                </range>
+            </ray>
+            <plugin filename="libgazebo_ros_range.so" name="gazebo_ros_range">
+                <gaussianNoise>0.005</gaussianNoise>
+                <alwaysOn>true</alwaysOn>
+                <updateRate>50</updateRate>
+                <topicName>sensor/ir_front_90</topicName>
+                <frameName>base_ir_front_90</frameName>
+                <radiation>INFRARED</radiation>
+                <fov>0.174533</fov>
+            </plugin>
+        </sensor>
+    </gazebo>
+    <gazebo reference="base_ir_front_135">
+        <sensor type="ray" name="TeraRanger">
+            <pose>0 0 0 0 0 0</pose>
+            <visualize>true</visualize>
+            <update_rate>15</update_rate>
+            <ray>
+                <scan>
+                    <horizontal>
+                    <samples>10</samples>
+                    <resolution>1</resolution>
+                    <min_angle>-0.14835</min_angle>
+                    <max_angle>0.14835</max_angle>
+                    </horizontal>
+                    <vertical>
+                    <samples>10</samples>
+                    <resolution>1</resolution>
+                    <min_angle>-0.14835</min_angle>
+                    <max_angle>0.14835</max_angle>
+                    </vertical>
+                </scan>
+                <range>
+                    <min>0.01</min>
+                    <max>7.5</max>
+                    <resolution>0.01</resolution>
+                </range>
+            </ray>
+            <plugin filename="libgazebo_ros_range.so" name="gazebo_ros_range">
+                <gaussianNoise>0.005</gaussianNoise>
+                <alwaysOn>true</alwaysOn>
+                <updateRate>50</updateRate>
+                <topicName>sensor/ir_front_135</topicName>
+                <frameName>base_ir_front_135</frameName>
+                <radiation>INFRARED</radiation>
+                <fov>0.174533</fov>
+            </plugin>
+        </sensor>
+    </gazebo>
+    <gazebo reference="base_ir_front_180">
+        <sensor type="ray" name="TeraRanger">
+            <pose>0 0 0 0 0 0</pose>
+            <visualize>true</visualize>
+            <update_rate>15</update_rate>
+            <ray>
+                <scan>
+                    <horizontal>
+                    <samples>10</samples>
+                    <resolution>1</resolution>
+                    <min_angle>-0.14835</min_angle>
+                    <max_angle>0.14835</max_angle>
+                    </horizontal>
+                    <vertical>
+                    <samples>10</samples>
+                    <resolution>1</resolution>
+                    <min_angle>-0.14835</min_angle>
+                    <max_angle>0.14835</max_angle>
+                    </vertical>
+                </scan>
+                <range>
+                    <min>0.01</min>
+                    <max>7.5</max>
+                    <resolution>0.01</resolution>
+                </range>
+            </ray>
+            <plugin filename="libgazebo_ros_range.so" name="gazebo_ros_range">
+                <gaussianNoise>0.005</gaussianNoise>
+                <alwaysOn>true</alwaysOn>
+                <updateRate>50</updateRate>
+                <topicName>sensor/ir_front_180</topicName>
+                <frameName>base_ir_front_180</frameName>
+                <radiation>INFRARED</radiation>
+                <fov>0.174533</fov>
+            </plugin>
+        </sensor>
+    </gazebo>
+    <gazebo reference="base_ir_front_225">
+        <sensor type="ray" name="TeraRanger">
+            <pose>0 0 0 0 0 0</pose>
+            <visualize>true</visualize>
+            <update_rate>15</update_rate>
+            <ray>
+                <scan>
+                    <horizontal>
+                    <samples>10</samples>
+                    <resolution>1</resolution>
+                    <min_angle>-0.14835</min_angle>
+                    <max_angle>0.14835</max_angle>
+                    </horizontal>
+                    <vertical>
+                    <samples>10</samples>
+                    <resolution>1</resolution>
+                    <min_angle>-0.14835</min_angle>
+                    <max_angle>0.14835</max_angle>
+                    </vertical>
+                </scan>
+                <range>
+                    <min>0.01</min>
+                    <max>7.5</max>
+                    <resolution>0.01</resolution>
+                </range>
+            </ray>
+            <plugin filename="libgazebo_ros_range.so" name="gazebo_ros_range">
+                <gaussianNoise>0.005</gaussianNoise>
+                <alwaysOn>true</alwaysOn>
+                <updateRate>50</updateRate>
+                <topicName>sensor/ir_front_225</topicName>
+                <frameName>base_ir_front_225</frameName>
+                <radiation>INFRARED</radiation>
+                <fov>0.174533</fov>
+            </plugin>
+        </sensor>
+    </gazebo>
+    <gazebo reference="base_ir_front_270">
+        <sensor type="ray" name="TeraRanger">
+            <pose>0 0 0 0 0 0</pose>
+            <visualize>true</visualize>
+            <update_rate>15</update_rate>
+            <ray>
+                <scan>
+                    <horizontal>
+                    <samples>10</samples>
+                    <resolution>1</resolution>
+                    <min_angle>-0.14835</min_angle>
+                    <max_angle>0.14835</max_angle>
+                    </horizontal>
+                    <vertical>
+                    <samples>10</samples>
+                    <resolution>1</resolution>
+                    <min_angle>-0.14835</min_angle>
+                    <max_angle>0.14835</max_angle>
+                    </vertical>
+                </scan>
+                <range>
+                    <min>0.01</min>
+                    <max>7.5</max>
+                    <resolution>0.01</resolution>
+                </range>
+            </ray>
+            <plugin filename="libgazebo_ros_range.so" name="gazebo_ros_range">
+                <gaussianNoise>0.005</gaussianNoise>
+                <alwaysOn>true</alwaysOn>
+                <updateRate>50</updateRate>
+                <topicName>sensor/ir_front_270</topicName>
+                <frameName>base_ir_front_270</frameName>
+                <radiation>INFRARED</radiation>
+                <fov>0.174533</fov>
+            </plugin>
+        </sensor>
+    </gazebo>
+    <gazebo reference="base_ir_front_315">
+        <sensor type="ray" name="TeraRanger">
+            <pose>0 0 0 0 0 0</pose>
+            <visualize>true</visualize>
+            <update_rate>15</update_rate>
+            <ray>
+                <scan>
+                    <horizontal>
+                    <samples>10</samples>
+                    <resolution>1</resolution>
+                    <min_angle>-0.14835</min_angle>
+                    <max_angle>0.14835</max_angle>
+                    </horizontal>
+                    <vertical>
+                    <samples>10</samples>
+                    <resolution>1</resolution>
+                    <min_angle>-0.14835</min_angle>
+                    <max_angle>0.14835</max_angle>
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