Commit message: 2v3423

File: hydrone_aerial_underwater_description/urdf/hydrone_aerial_underwater_aerial.gazebo.xacro (robot description, xacro)
@@ -11,4 +11,5 @@
     <!-- <xacro:property name="volume" value="0.00001"/> -->
     <xacro:property name="volume" value="0.001"/>
+    <!-- <xacro:property name="volume" value="0.0001"/> -->
     <xacro:property name="M_PI" value="3.1415926535897931" />
     <xacro:macro name="hydrone_aerial_underwater_hydro_model" params="namespace">
@@ -100,5 +101,5 @@
         <sensor type="ray" name="VLP-16-VLP16-Simplified">
         <pose>0 0 0 0 0 0</pose>
-        <visualize>true</visualize>
+        <visualize>false</visualize>
         <update_rate>5</update_rate>
         <ray>

Commit message: 23v423

File: hydrone_aerial_underwater_description/urdf/hydrone_aerial_underwater_aerial.gazebo.xacro (robot description, xacro)
@@ -10,6 +10,6 @@
     <!-- <xacro:property name="volume" value="1.83826"/> -->
     <!-- <xacro:property name="volume" value="0.00001"/> -->
-    <xacro:property name="volume" value="0.001"/>
-    <!-- <xacro:property name="volume" value="0.0001"/> -->
+    <!-- <xacro:property name="volume" value="0.001"/> -->
+    <xacro:property name="volume" value="0.0001"/>
     <xacro:property name="M_PI" value="3.1415926535897931" />
     <xacro:macro name="hydrone_aerial_underwater_hydro_model" params="namespace">

Commit message: v3423

File: hydrone_aerial_underwater_description/urdf/hydrone_aerial_underwater_aerial.gazebo.xacro (robot description, xacro)
@@ -10,6 +10,7 @@
     <!-- <xacro:property name="volume" value="1.83826"/> -->
     <!-- <xacro:property name="volume" value="0.00001"/> -->
-    <!-- <xacro:property name="volume" value="0.001"/> -->
-    <xacro:property name="volume" value="0.0001"/>
+    <xacro:property name="volume" value="0.001"/>
+    <!-- <xacro:property name="volume" value="0.0001"/> -->
+    <!-- <xacro:property name="volume" value="0.00005"/> -->
     <xacro:property name="M_PI" value="3.1415926535897931" />
     <xacro:macro name="hydrone_aerial_underwater_hydro_model" params="namespace">

Commit message: 23v423

File: hydrone_aerial_underwater_description/urdf/hydrone_aerial_underwater_aerial.gazebo.xacro (robot description, xacro)
@@ -10,7 +10,7 @@
     <!-- <xacro:property name="volume" value="1.83826"/> -->
     <!-- <xacro:property name="volume" value="0.00001"/> -->
-    <xacro:property name="volume" value="0.001"/>
+    <!-- <xacro:property name="volume" value="0.001"/> -->
     <!-- <xacro:property name="volume" value="0.0001"/> -->
-    <!-- <xacro:property name="volume" value="0.00005"/> -->
+    <xacro:property name="volume" value="0.00005"/>
     <xacro:property name="M_PI" value="3.1415926535897931" />
     <xacro:macro name="hydrone_aerial_underwater_hydro_model" params="namespace">

Commit message: 2v342v3

File: hydrone_aerial_underwater_description/urdf/hydrone_aerial_underwater_aerial.gazebo.xacro (robot description, xacro)
@@ -11,6 +11,6 @@
     <!-- <xacro:property name="volume" value="0.00001"/> -->
     <!-- <xacro:property name="volume" value="0.001"/> -->
-    <xacro:property name="volume" value="0.0001"/>
-    <!-- <xacro:property name="volume" value="0.00005"/> -->
+    <!-- <xacro:property name="volume" value="0.0001"/> -->
+    <xacro:property name="volume" value="0.00005"/>
     <xacro:property name="M_PI" value="3.1415926535897931" />
     <xacro:macro name="hydrone_aerial_underwater_hydro_model" params="namespace">

Commit message: 2v342v3

File: hydrone_aerial_underwater_description/urdf/hydrone_aerial_underwater_aerial.gazebo.xacro (robot description, xacro)
@@ -11,6 +11,6 @@
     <!-- <xacro:property name="volume" value="0.00001"/> -->
     <!-- <xacro:property name="volume" value="0.001"/> -->
-    <!-- <xacro:property name="volume" value="0.0001"/> -->
-    <xacro:property name="volume" value="0.00005"/>
+    <xacro:property name="volume" value="0.0001"/>
+    <!-- <xacro:property name="volume" value="0.00005"/> -->
     <xacro:property name="M_PI" value="3.1415926535897931" />
     <xacro:macro name="hydrone_aerial_underwater_hydro_model" params="namespace">
